Commit message: collision

File: src/clase4/robots/mycobot_320_m5_2022/mycobot_320_m5_2022.urdf (robot description, URDF)
Before this commit: robot myCobot320, 7 links, 6 joints
Links:
- link link5: geometry collision box size=0.103 0.059 0.080; visual mesh filename=package://clase4/robots/mycobot_320_m5_2022/link5.dae
